Commit message: rename link

File: src/tstar_description/urdf/gq7.urdf.xacro (robot description, xacro)
@@ -14,5 +14,5 @@
       </visual>
     </link>
-    <link name="${name}">
+    <link name="${name}_imu_link">
     </link>
     <!-- This joint handles the center of the GQ7, but measurements will not be produced WRT to this, it is just easier to place on robots -->
@@ -25,5 +25,5 @@
     <joint name="${name}_joint" type="fixed">
       <parent link="${name}_center" />
-      <child link="${name}" />
+      <child link="${name}_imu_link" />
       <origin xyz="-0.0222 -0.015585 0.00737" rpy="0 0 0" />
     </joint>

File: src/tstar_description/urdf/tartanstar.urdf.xacro (robot description, xacro)
@@ -64,5 +64,5 @@
   </link>
   <link
-    name="gps">
+    name="gq7_gnss_1_antenna_link">
     <inertial>
       <origin
@@ -112,5 +112,5 @@
       link="base_link" />
     <child
-      link="gps" />
+      link="gq7_gnss_1_antenna_link" />
     <axis
       xyz="0 0 0" />
